Commit message: v3

File: urdf/mobile_base.xacro (robot description, xacro)
@@ -46,5 +46,5 @@
                     <cylinder radius="${wheel_radius}" length="${wheel_length}"/>
                 </geometry>
-                <origin xyz="0 0 0" rpy="${pi/2.0} 0 0"/>
+                <origin xyz="0 0 0" rpy="0 0 0"/>
                 <material name ="grey"/>
             </visual>
@@ -54,5 +54,5 @@
                     <cylinder radius="${wheel_radius}" length="${wheel_length}"/>
                 </geometry>
-                <origin xyz="0 0 0" rpy="${pi/2.0} 0 0"/>
+                <origin xyz="0 0 0" rpy="0 0 0"/>
             </collision>
         </link>
@@ -95,9 +95,9 @@
         <origin xyz="0 0 ${wheel_radius}" rpy="0 0 0"/>
     </joint>
-    <joint name="base_right_wheel_joint" type="continuous">
+    <joint name="right_wheel_joint" type="continuous">
         <parent link="base_link"/>
         <child link="right_wheel_link"/>
-        <origin xyz="${-base_length / 4.0} ${-((base_width / 2.0) + (wheel_length/2.0))} 0" rpy="0 0 0"/>
-        <axis xyz="0 1 0"/>
+        <origin xyz="${-base_length / 4.0} ${-((base_width / 2.0) + (wheel_length/2.0))} 0" rpy="${pi/2} 0 0"/>
+        <axis xyz="0 0 1"/>
         <limit velocity="100" effort="100"/>
     </joint>
@@ -105,5 +105,5 @@
         <parent link="base_link"/>
         <child link="laser_frame"/>
-        <origin xyz="0.0 0.0 0.05" rpy="3.14 0 3.14"/>
+        <origin xyz="0.0 0.0 0.2" rpy="0 0 0"/>
         <axis xyz="0 0 0"/>
         <limit velocity="100" effort="100"/>
@@ -116,9 +116,9 @@
         <limit velocity="100" effort="100"/>
     </joint>
-    <joint name="base_left_wheel_joint" type="continuous">
+    <joint name="left_wheel_joint" type="continuous">
         <parent link="base_link"/>
         <child link="left_wheel_link"/>
-        <origin xyz="${-base_length / 4.0} ${(base_width / 2.0) + (wheel_length/2.0)} 0" rpy="0 0 0"/>
-        <axis xyz="0 1 0"/>
+        <origin xyz="${-base_length / 4.0} ${(base_width / 2.0) + (wheel_length/2.0)} 0" rpy="-${pi/2} 0 0"/>
+        <axis xyz="0 0 1"/>
         <limit velocity="100" effort="100"/>
     </joint>

File: urdf/my_robot.urdf.xacro (robot description, xacro)
@@ -3,3 +3,4 @@
     <xacro:include filename="common_properties.xacro"/>
     <xacro:include filename="mobile_base.xacro"/>
+    <xacro:include filename="ros2_control.xacro"/>
 </robot>
